File: mcuheaders.kicad_sch (KiCad schematic)
At the start: 4 parts, among them J1 Left_02x24, J2 Right Header, J3 Right_02x24, J4 Left Header

Commit message: sync from JLCPCB mcuheaders.kicad_sch
Parts:
- J1, J3: symbol Connector_Generic:Conn_02x24_Odd_Even -> EggClassifier:Conn_02x24_Odd_Even
- J2, J4: symbol LM2676S-3.3_NOPB:Conn_02x22_Odd_Even -> EggClassifier:Conn_02x22_Odd_Even
Changed lines of the file:
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@@
 	(paper "A4")
 	(junction
-		(at 43.18 100.33)
-		(diameter 0)
-		(color 0 0 0 0)
-	)
-	(junction
 		(at 171.45 26.67)
 		(diameter 0)
@@
 		(color 0 0 0 0)
 	)
-	(junction
-		(at 90.17 105.41)
-		(diameter 0)
-		(color 0 0 0 0)
-	)
 	(no_connect
 		(at 71.12 107.95)
@@
 	(wire
 		(pts
-			(xy 43.18 100.33) (xy 39.37 100.33)
-		)
-		(stroke
-			(width 0)
-			(type default)
-		)
-	)
-	(wire
-		(pts
 			(xy 77.47 120.65) (xy 71.12 120.65)
 		)
@@
 	(wire
 		(pts
-			(xy 90.17 105.41) (xy 91.44 105.41)
-		)
-		(stroke
-			(width 0)
-			(type default)
-		)
-	)
-	(wire
-		(pts
 			(xy 77.47 153.67) (xy 71.12 153.67)
 		)
@@
 	(wire
 		(pts
-			(xy 58.42 100.33) (xy 43.18 100.33)
+			(xy 39.37 100.33) (xy 58.42 100.33)
 		)
 		(stroke
@@
 	)
 	(symbol
-		(lib_id "LM2676S-3.3_NOPB:Conn_02x22_Odd_Even")
+		(lib_id "EggClassifier:Conn_02x22_Odd_Even")
 		(at 63.5 125.73 0)
 		(unit 1)
@@
 	)
 	(symbol
-		(lib_id "LM2676S-3.3_NOPB:PWR_FLAG")
-		(at 91.44 105.41 270)
-		(unit 1)
-		(exclude_from_sim no)
-		(in_bom yes)
-		(on_board yes)
-		(dnp no)
-		(fields_autoplaced yes)
-		(property "Reference" "#FLG02"
-			(at 93.345 105.41 0)
-			(effects
-				(font
-					(size 1.27 1.27)
-				)
-				(hide yes)
-			)
-		)
-		(property "Value" "PWR_FLAG"
-			(at 95.25 105.4099 90)
-			(effects
-				(font
-					(size 1.27 1.27)
-				)
-				(justify left)
-			)
-		)
-		(property "Footprint" ""
-			(at 91.44 105.41 0)
-			(effects
-				(font
-					(size 1.27 1.27)
-				)
-				(hide yes)
-			)
-		)
-		(property "Datasheet" "~"
-			(at 91.44 105.41 0)
-			(effects
-				(font
-					(size 1.27 1.27)
-				)
-				(hide yes)
-			)
-		)
-		(property "Description" "Special symbol for telling ERC where power comes from"
-			(at 91.44 105.41 0)
-			(effects
-				(font
-					(size 1.27 1.27)
-				)
-				(hide yes)
-			)
-		)
-		(pin "1"
-		)
-		(instances
-			(project "EggClassifier"
-				(path "/1c72d2eb-7fb1-49fe-a026-e817f5a7ec43/a876cc3c-46f3-4b62-bd95-490c4538aae6"
-					(reference "#FLG02")
-					(unit 1)
-				)
-			)
-		)
-	)
-	(symbol
 		(lib_id "LM2676S-3.3_NOPB:GND")
 		(at 187.96 104.14 0)
@@
 	)
 	(symbol
-		(lib_id "Connector_Generic:Conn_02x24_Odd_Even")
+		(lib_id "EggClassifier:Conn_02x24_Odd_Even")
 		(at 161.29 54.61 0)
 		(unit 1)
@@
 	)
 	(symbol
-		(lib_id "LM2676S-3.3_NOPB:PWR_FLAG")
-		(at 43.18 100.33 0)
-		(unit 1)
-		(exclude_from_sim no)
-		(in_bom yes)
-		(on_board yes)
-		(dnp no)
-		(fields_autoplaced yes)
-		(property "Reference" "#FLG01"
-			(at 43.18 98.425 0)
-			(effects
-				(font
-					(size 1.27 1.27)
-				)
-				(hide yes)
-			)
-		)
-		(property "Value" "PWR_FLAG"
-			(at 43.18 95.25 0)
-			(effects
-				(font
-					(size 1.27 1.27)
-				)
-			)
-		)
-		(property "Footprint" ""
-			(at 43.18 100.33 0)
-			(effects
-				(font
-					(size 1.27 1.27)
-				)
-				(hide yes)
-			)
-		)
-		(property "Datasheet" "~"
-			(at 43.18 100.33 0)
-			(effects
-				(font
-					(size 1.27 1.27)
-				)
-				(hide yes)
-			)
-		)
-		(property "Description" "Special symbol for telling ERC where power comes from"
-			(at 43.18 100.33 0)
-			(effects
-				(font
-					(size 1.27 1.27)
-				)
-				(hide yes)
-			)
-		)
-		(pin "1"
-		)
-		(instances
-			(project "EggClassifier"
-				(path "/1c72d2eb-7fb1-49fe-a026-e817f5a7ec43/a876cc3c-46f3-4b62-bd95-490c4538aae6"
-					(reference "#FLG01")
-					(unit 1)
-				)
-			)
-		)
-	)
-	(symbol
-		(lib_id "Connector_Generic:Conn_02x24_Odd_Even")
+		(lib_id "EggClassifier:Conn_02x24_Odd_Even")
 		(at 63.5 54.61 0)
 		(unit 1)
@@
 	)
 	(symbol
-		(lib_id "LM2676S-3.3_NOPB:Conn_02x22_Odd_Even")
+		(lib_id "EggClassifier:Conn_02x22_Odd_Even")
 		(at 161.29 127 0)
 		(unit 1)

Commit message: update footprints
Parts:
- J1, J3: footprint Connector_PinHeader_2.54mm:PinHeader_2x24_P2.54mm_Vertical -> EggClassifier:PinHeader_2x24_P2.54mm_Vertical
- J2, J4: footprint Connector_PinHeader_2.54mm:PinHeader_2x22_P2.54mm_Vertical -> EggClassifier:PinHeader_2x22_P2.54mm_Vertical
Changed lines of the file:
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@@
 			)
 		)
-		(property "Footprint" "Connector_PinHeader_2.54mm:PinHeader_2x22_P2.54mm_Vertical"
+		(property "Footprint" "EggClassifier:PinHeader_2x22_P2.54mm_Vertical"
 			(at 63.5 125.73 0)
 			(effects
@@
 			)
 		)
-		(property "Footprint" "Connector_PinHeader_2.54mm:PinHeader_2x24_P2.54mm_Vertical"
+		(property "Footprint" "EggClassifier:PinHeader_2x24_P2.54mm_Vertical"
 			(at 161.29 54.61 0)
 			(effects
@@
 			)
 		)
-		(property "Footprint" "Connector_PinHeader_2.54mm:PinHeader_2x24_P2.54mm_Vertical"
+		(property "Footprint" "EggClassifier:PinHeader_2x24_P2.54mm_Vertical"
 			(at 63.5 54.61 0)
 			(effects
@@
 			)
 		)
-		(property "Footprint" "Connector_PinHeader_2.54mm:PinHeader_2x22_P2.54mm_Vertical"
+		(property "Footprint" "EggClassifier:PinHeader_2x22_P2.54mm_Vertical"
 			(at 161.29 127 0)
 			(effects
