File: baseboard.kicad_sch (KiCad schematic)
At the start: 50 parts, among them J10 LCD_CHAR, J11 SERVO2, J12 BME280, J13 UART1, J14 FAN, J15 UART2, J16 AS7265X, J17 TFT_SPI, J5 POWER, J6 DCMI_CAMERA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

Commit message: snapshot prior to merge
Parts:
- C1: symbol Library:C_Polarized -> EggClassifier:C_Polarized
- C10, C11, C2, C5, C6, C7, C8, C9: symbol Library:C -> EggClassifier:C
- C3, C4: symbol Library:C_Polarized_US -> EggClassifier:C_Polarized_US
- D1: symbol PCM_Diode_Schottky_AKL:SS56BF -> EggClassifier:SS56BF
- D2, D3, D4: symbol Library:SS36 -> EggClassifier:SS36
- D5: symbol Library:LED -> EggClassifier:LED
- H1, H2, H3, H4: symbol Library:Mounting Hole, 3mm, Via Stiched -> EggClassifier:Mounting Hole, 3mm, Via Stiched
- J10, J12, J16, J5: symbol Library:Conn_01x04 -> EggClassifier:Conn_01x04
- J11, J13, J14, J15, J8, J9: symbol Library:Conn_01x03 -> EggClassifier:Conn_01x03
- J17: symbol Library:Conn_01x15 -> EggClassifier:Conn_01x15
- J6: symbol Library:Conn_02x09_Odd_Even -> EggClassifier:Conn_02x09_Odd_Even
- J7: symbol Library:Conn_02x05_Odd_Even -> EggClassifier:Conn_02x05_Odd_Even
- L1: symbol Library:CDRH104RNP-330NC -> EggClassifier:CDRH104RNP-330NC
- Q1, Q2, Q3: symbol Library:BCP56 -> EggClassifier:BCP56
- R1, R10, R11, R2, R3, R4, R5, R6, R7, R8, R9: symbol Library:R_Small -> EggClassifier:R_Small
- U1: symbol Library:LM2676S-3.3_NOPB -> EggClassifier:LM2676S-3.3_NOPB
- U2: symbol Library:AMS1117-3.3 -> EggClassifier:AMS1117-3.3

Commit message: sync from JLCPCB
Changed lines of the file:
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@@
 	)
 	(junction
+		(at 146.05 124.46)
+		(diameter 0)
+		(color 0 0 0 0)
+	)
+	(junction
 		(at 109.22 38.1)
 		(diameter 0)
@@
 	(wire
 		(pts
+			(xy 146.05 124.46) (xy 147.32 124.46)
+		)
+		(stroke
+			(width 0)
+			(type default)
+		)
+	)
+	(wire
+		(pts
 			(xy 67.31 59.69) (xy 58.42 59.69)
 		)
@@
 	(wire
 		(pts
+			(xy 146.05 123.19) (xy 146.05 124.46)
+		)
+		(stroke
+			(width 0)
+			(type default)
+		)
+	)
+	(wire
+		(pts
 			(xy 168.91 135.89) (xy 166.37 135.89)
 		)
@@
 		(dnp no)
 		(fields_autoplaced yes)
-		(property "Reference" "#FLG01"
+		(property "Reference" "#FLG0101"
 			(at 173.99 159.385 0)
 			(effects
@@
 			(project ""
 				(path "/1c72d2eb-7fb1-49fe-a026-e817f5a7ec43/16aff487-3924-4be3-b176-d1fab0e3868e"
-					(reference "#FLG01")
+					(reference "#FLG0101")
 					(unit 1)
 				)
@@
 	(symbol
 		(lib_id "LM2676S-3.3_NOPB:+5V")
-		(at 146.05 124.46 0)
+		(at 146.05 123.19 0)
 		(unit 1)
 		(exclude_from_sim no)
@@
 		(fields_autoplaced yes)
 		(property "Reference" "#PWR039"
-			(at 146.05 128.27 0)
+			(at 146.05 127 0)
 			(effects
 				(font
@@
 		)
 		(property "Value" "+5V"
-			(at 146.05 119.38 0)
+			(at 146.05 118.11 0)
 			(effects
 				(font
@@
 		)
 		(property "Footprint" ""
-			(at 146.05 124.46 0)
+			(at 146.05 123.19 0)
 			(effects
 				(font
@@
 		)
 		(property "Datasheet" ""
-			(at 146.05 124.46 0)
+			(at 146.05 123.19 0)
 			(effects
 				(font
@@
 		)
 		(property "Description" "Power symbol creates a global label with name \"+5V\""
-			(at 146.05 124.46 0)
+			(at 146.05 123.19 0)
 			(effects
 				(font
@@
 					(unit 1)
 				)
+			)
+		)
+	)
+	(symbol
+		(lib_id "LM2676S-3.3_NOPB:PWR_FLAG")
+		(at 147.32 124.46 270)
+		(unit 1)
+		(exclude_from_sim no)
+		(in_bom yes)
+		(on_board yes)
+		(dnp no)
+		(fields_autoplaced yes)
+		(property "Reference" "#FLG01"
+			(at 149.225 124.46 0)
+			(effects
+				(font
+					(size 1.27 1.27)
+				)
+				(hide yes)
+			)
+		)
+		(property "Value" "PWR_FLAG"
+			(at 151.13 124.4599 90)
+			(effects
+				(font
+					(size 1.27 1.27)
+				)
+				(justify left)
+			)
+		)
+		(property "Footprint" ""
+			(at 147.32 124.46 0)
+			(effects
+				(font
+					(size 1.27 1.27)
+				)
+				(hide yes)
+			)
+		)
+		(property "Datasheet" "~"
+			(at 147.32 124.46 0)
+			(effects
+				(font
+					(size 1.27 1.27)
+				)
+				(hide yes)
+			)
+		)
+		(property "Description" "Special symbol for telling ERC where power comes from"
+			(at 147.32 124.46 0)
+			(effects
+				(font
+					(size 1.27 1.27)
+				)
+				(hide yes)
+			)
+		)
+		(pin "1"
+		)
+		(instances
+			(project ""
+				(path "/1c72d2eb-7fb1-49fe-a026-e817f5a7ec43/16aff487-3924-4be3-b176-d1fab0e3868e"
+					(reference "#FLG01")
+					(unit 1)
+				)
