File: devebox.kicad_sch (KiCad schematic)
At the start: 27 parts, among them J1 ST-LINK, J2 USB_A, SW1 RESET SW, U3 STM32H743VITx, U4 W25Q128, Y1 25MHZ

Commit message: final version of 80mmx140mm PCB
Parts:
- Y1: footprint EggClassifier:Oscillator_SMD_Abracon_ASV-4Pin_7.0x5.1mm_HandSoldering -> EggClassifier:Oscillator_SMD_EuroQuartz_XO91-4Pin_7.0x5.0mm_HandSoldering
Changed lines of the file:
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@@
 			)
 		)
-		(property "Footprint" "EggClassifier:Oscillator_SMD_Abracon_ASV-4Pin_7.0x5.1mm_HandSoldering"
+		(property "Footprint" "EggClassifier:Oscillator_SMD_EuroQuartz_XO91-4Pin_7.0x5.0mm_HandSoldering"
 			(at 41.91 62.23 0)
 			(effects

Commit message: Snapshot prior to making JLC version
Parts:
- Y1: footprint EggClassifier:Oscillator_SMD_EuroQuartz_XO91-4Pin_7.0x5.0mm_HandSoldering -> Oscillator:Oscillator_SMD_SeikoEpson_SG8002CA-4Pin_7.0x5.0mm; symbol EggClassifier:ASCO -> Oscillator:SG-7050CAN
Changed lines of the file:
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@@
 	(wire
 		(pts
+			(xy 46.99 53.34) (xy 60.96 53.34)
+		)
+		(stroke
+			(width 0)
+			(type default)
+		)
+	)
+	(wire
+		(pts
 			(xy 257.81 82.55) (xy 257.81 83.82)
 		)
@@
 	(wire
 		(pts
-			(xy 49.53 53.34) (xy 60.96 53.34)
-		)
-		(stroke
-			(width 0)
-			(type default)
-		)
-	)
-	(wire
-		(pts
 			(xy 25.4 43.18) (xy 25.4 45.72)
 		)
@@
 	(wire
 		(pts
-			(xy 26.67 53.34) (xy 29.21 53.34)
+			(xy 29.21 53.34) (xy 31.75 53.34)
 		)
 		(stroke
@@
 	)
 	(symbol
-		(lib_id "EggClassifier:ASCO")
+		(lib_id "Oscillator:SG-7050CAN")
 		(at 39.37 53.34 0)
 		(unit 1)
@@
 			)
 		)
-		(property "Footprint" "EggClassifier:Oscillator_SMD_EuroQuartz_XO91-4Pin_7.0x5.0mm_HandSoldering"
-			(at 41.91 62.23 0)
+		(property "Footprint" "Oscillator:Oscillator_SMD_SeikoEpson_SG8002CA-4Pin_7.0x5.0mm"
+			(at 57.15 62.23 0)
 			(effects
 				(font
@@
 			)
 		)
-		(property "Datasheet" "https://abracon.com/Oscillators/ASCO.pdf"
-			(at 33.655 50.165 0)
+		(property "Datasheet" "https://support.epson.biz/td/api/doc_check.php?dl=brief_SG7050CAN&lang=en"
+			(at 36.83 53.34 0)
 			(effects
 				(font
@@
 			)
 		)
-		(property "Description" "Crystal Clock Oscillator, Abracon ASCO"
+		(property "Description" "CMOS Clock Oscillator 1 to 75 MHz"
 			(at 39.37 53.34 0)
 			(effects
@@
 	(symbol
 		(lib_id "LM2676S-3.3_NOPB:+3.3V")
-		(at 26.67 53.34 90)
+		(at 29.21 53.34 90)
 		(unit 1)
 		(exclude_from_sim no)
@@
 		(dnp no)
 		(property "Reference" "#PWR02"
-			(at 30.48 53.34 0)
+			(at 33.02 53.34 0)
 			(effects
 				(font
@@
 		)
 		(property "Value" "+3.3V"
-			(at 23.876 53.594 90)
+			(at 26.416 53.594 90)
 			(effects
 				(font
@@
 		)
 		(property "Footprint" ""
-			(at 26.67 53.34 0)
+			(at 29.21 53.34 0)
 			(effects
 				(font
@@
 		)
 		(property "Datasheet" ""
-			(at 26.67 53.34 0)
+			(at 29.21 53.34 0)
 			(effects
 				(font
@@
 		)
 		(property "Description" "Power symbol creates a global label with name \"+3.3V\""
-			(at 26.67 53.34 0)
+			(at 29.21 53.34 0)
 			(effects
 				(font

Commit message: end of day snapshot
Parts:
- J1, J2, SW1: now left out of the parts list
Changed lines of the file:
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@@
 		(unit 1)
 		(exclude_from_sim no)
-		(in_bom yes)
+		(in_bom no)
 		(on_board yes)
 		(dnp no)
@@
 		(unit 1)
 		(exclude_from_sim no)
-		(in_bom yes)
+		(in_bom no)
 		(on_board yes)
 		(dnp no)
@@
 		(unit 1)
 		(exclude_from_sim no)
-		(in_bom yes)
-		(on_board yes)
-		(dnp no)
+		(in_bom no)
+		(on_board yes)
+		(dnp no)
